Commit message: add .gitignore

File: model/franka_panda_urdf/robots/panda_arm.urdf (robot description, URDF)
Before this commit: robot panda, 10 links, 9 joints
Links:
- removed link ee_center_body
- removed link hand
- link link0: mass None -> 0.629769
Joints:
- removed joint joint8
- removed joint joint9
- joint joint6: limit lower=-0.0175 upper=3.7525 effort=12 velocity=2.6100 -> lower=-3.7525 upper=3.7525 effort=12 velocity=2.6100
